Commit message: Align robot geometry and sensor fusion frames

File: src/bagheera_base/urdf/bagheera.urdf.xacro (robot description, xacro)
@@ -2,15 +2,16 @@
 <robot name="bagheera" xmlns:xacro="http://www.ros.org/wiki/xacro">
   <!-- REP-103: x forward, y left, z up. base_footprint lies on the floor. -->
-  <xacro:arg name="chassis_length" default="0.60"/>
-  <xacro:arg name="chassis_width" default="0.40"/>
+  <xacro:arg name="chassis_length" default="0.51"/>
+  <xacro:arg name="chassis_width" default="0.34"/>
   <xacro:arg name="chassis_height" default="0.19"/>
-  <xacro:arg name="chassis_center_x" default="0.18"/>
+  <xacro:arg name="chassis_center_x" default="0.075"/>
   <xacro:arg name="chassis_mass_kg" default="8.76"/>
   <xacro:arg name="wheel_radius" default="0.04475"/>
   <xacro:arg name="wheel_width" default="0.04"/>
-  <xacro:arg name="wheel_track" default="0.325"/>
+  <xacro:arg name="wheel_track" default="0.32"/>
+  <xacro:arg name="axle_x" default="0.0"/>
   <xacro:arg name="caster_radius" default="0.03"/>
   <xacro:arg name="caster_track" default="0.36"/>
-  <xacro:arg name="imu_x" default="0.18"/>
+  <xacro:arg name="imu_x" default="0.08"/>
   <xacro:arg name="imu_y" default="0.0"/>
   <xacro:arg name="imu_z" default="0.095"/>
@@ -18,12 +19,12 @@
   <xacro:arg name="imu_pitch" default="0.0"/>
   <xacro:arg name="imu_yaw" default="0.0"/>
-  <xacro:arg name="lidar_x" default="0.0"/>
+  <xacro:arg name="lidar_x" default="0.08"/>
   <xacro:arg name="lidar_y" default="0.0"/>
   <xacro:arg name="lidar_z" default="0.30"/>
   <xacro:arg name="lidar_yaw" default="0.0"/>
-  <xacro:arg name="optical_flow_x" default="0.0"/>
+  <xacro:arg name="optical_flow_x" default="0.08"/>
   <xacro:arg name="optical_flow_y" default="0.0"/>
   <xacro:arg name="optical_flow_z" default="0.04525"/>
-  <xacro:arg name="camera_x" default="0.48"/>
+  <xacro:arg name="camera_x" default="0.33"/>
   <xacro:arg name="camera_y" default="0.0"/>
   <xacro:arg name="camera_z" default="0.12"/>
@@ -54,8 +55,8 @@
       <origin xyz="$(arg chassis_center_x) 0 ${float($(arg chassis_height))/2.0}"/>
       <mass value="$(arg chassis_mass_kg)"/>
-      <inertia ixx="0.144" ixy="0" ixz="0" iyy="0.289" iyz="0" izz="0.380"/>
+      <inertia ixx="0.111" ixy="0" ixz="0" iyy="0.216" iyz="0" izz="0.274"/>
     </inertial>
   </link>
-  <xacro:macro name="fixed_wheel" params="name x y radius width">
+  <xacro:macro name="fixed_wheel" params="name parent x y radius width">
     <link name="${name}_link">
       <visual>
@@ -70,12 +71,17 @@
     </link>
     <joint name="${name}_joint" type="fixed">
-      <parent link="base_link"/><child link="${name}_link"/>
+      <parent link="${parent}"/><child link="${name}_link"/>
       <origin xyz="${x} ${y} 0"/>
     </joint>
   </xacro:macro>
-  <xacro:fixed_wheel name="left_wheel" x="0" y="${float($(arg wheel_track))/2.0}" radius="$(arg wheel_radius)" width="$(arg wheel_width)"/>
-  <xacro:fixed_wheel name="right_wheel" x="0" y="${-float($(arg wheel_track))/2.0}" radius="$(arg wheel_radius)" width="$(arg wheel_width)"/>
-  <xacro:fixed_wheel name="front_left_caster" x="${caster_x}" y="${float($(arg caster_track))/2.0}" radius="$(arg caster_radius)" width="0.03"/>
-  <xacro:fixed_wheel name="front_right_caster" x="${caster_x}" y="${-float($(arg caster_track))/2.0}" radius="$(arg caster_radius)" width="0.03"/>
+  <link name="base_axle"/>
+  <joint name="base_axle_joint" type="fixed">
+    <parent link="base_link"/><child link="base_axle"/>
+    <origin xyz="$(arg axle_x) 0 0" rpy="0 0 0"/>
+  </joint>
+  <xacro:fixed_wheel name="left_wheel" parent="base_axle" x="0" y="${float($(arg wheel_track))/2.0}" radius="$(arg wheel_radius)" width="$(arg wheel_width)"/>
+  <xacro:fixed_wheel name="right_wheel" parent="base_axle" x="0" y="${-float($(arg wheel_track))/2.0}" radius="$(arg wheel_radius)" width="$(arg wheel_width)"/>
+  <xacro:fixed_wheel name="front_left_caster" parent="base_link" x="${caster_x}" y="${float($(arg caster_track))/2.0}" radius="$(arg caster_radius)" width="0.03"/>
+  <xacro:fixed_wheel name="front_right_caster" parent="base_link" x="${caster_x}" y="${-float($(arg caster_track))/2.0}" radius="$(arg caster_radius)" width="0.03"/>
   <link name="imu_link"/>
   <joint name="imu_joint" type="fixed">
